File: supply.sch (KiCad schematic (older format))
At the start: 42 parts, among them Q1 Q_NMOS_GDS, Q2 Q_NMOS_GDS, Q3 Q_NMOS_GDS, U4 BTS50085-1TMA, U5 LM5022MM, U6 TSR_1-24120, U7 TSR_1-2450

Commit message: started assigning footprints
Parts:
- C12, C13, C20, C25, C27, C29, C30: footprint (none) -> Capacitor_THT:CP_Radial_D16.0mm_P7.50mm
- C14, C15, C16, C17, C18, C21, C22, C23, C28: footprint (none) -> Capacitor_SMD:C_0603_1608Metric
- C19: footprint (none) -> Capacitor_SMD:CP_Elec_4x3.9
- C24, C31: footprint (none) -> Capacitor_SMD:C_1206_3216Metric
- D2: footprint (none) -> Diode_SMD:D_1206_3216Metric
- Q1, Q2: footprint (none) -> FE Footprints:SOT-23
- Q3: footprint (none) -> FE Footprints:TO-252
- R18, R19, R20, R21, R22, R23, R24, R25, R27, R28, R29: footprint (none) -> Resistor_SMD:R_0603_1608Metric
- R26: footprint (none) -> Resistor_SMD:R_1206_3216Metric
- TP7: footprint (none) -> TestPoint:TestPoint_Pad_2.5x2.5mm
Changed lines of the file:
@@
 F 0 "R20" H 4300 1500 50  0000 R CNN
 F 1 "10K" H 4350 1600 50  0000 R CNN
-F 2 "" V 4080 1550 50  0001 C CNN
+F 2 "Resistor_SMD:R_0603_1608Metric" V 4080 1550 50  0001 C CNN
 F 3 "~" H 4150 1550 50  0001 C CNN
 	1    4150 1550
@@
 F 0 "R21" H 4300 2400 50  0000 R CNN
 F 1 "470" H 4400 2500 50  0000 R CNN
-F 2 "" V 4080 2450 50  0001 C CNN
+F 2 "Resistor_SMD:R_0603_1608Metric" V 4080 2450 50  0001 C CNN
 F 3 "~" H 4150 2450 50  0001 C CNN
 	1    4150 2450
@@
 F 0 "R22" H 4500 2300 50  0000 R CNN
 F 1 "86K" H 4350 2300 50  0000 R CNN
-F 2 "" V 4330 2450 50  0001 C CNN
+F 2 "Resistor_SMD:R_0603_1608Metric" V 4330 2450 50  0001 C CNN
 F 3 "~" H 4400 2450 50  0001 C CNN
 	1    4400 2450
@@
 F 0 "C15" H 4765 2496 50  0000 L CNN
 F 1 "10nF" H 4765 2405 50  0000 L CNN
-F 2 "" H 4688 2300 50  0001 C CNN
+F 2 "Capacitor_SMD:C_0603_1608Metric" H 4688 2300 50  0001 C CNN
 F 3 "~" H 4650 2450 50  0001 C CNN
 	1    4650 2450
@@
 F 0 "Q3" H 6855 1596 50  0000 L CNN
 F 1 "Q_NMOS_GDS" H 6855 1505 50  0000 L CNN
-F 2 "" H 6850 1650 50  0001 C CNN
+F 2 "FE Footprints:TO-252" H 6850 1650 50  0001 C CNN
 F 3 "~" H 6650 1550 50  0001 C CNN
 	1    6650 1550
@@
 F 0 "R23" V 6007 1550 50  0000 C CNN
 F 1 "10" V 5916 1550 50  0000 C CNN
-F 2 "" V 5730 1550 50  0001 C CNN
+F 2 "Resistor_SMD:R_0603_1608Metric" V 5730 1550 50  0001 C CNN
 F 3 "~" H 5800 1550 50  0001 C CNN
 	1    5800 1550
@@
 F 0 "R26" H 6820 2196 50  0000 L CNN
 F 1 "40m" H 6820 2105 50  0000 L CNN
-F 2 "" V 6680 2150 50  0001 C CNN
+F 2 "Resistor_SMD:R_1206_3216Metric" V 6680 2150 50  0001 C CNN
 F 3 "~" H 6750 2150 50  0001 C CNN
 	1    6750 2150
@@
 F 0 "R25" V 6343 1900 50  0000 C CNN
 F 1 "100" V 6434 1900 50  0000 C CNN
-F 2 "" V 6480 1900 50  0001 C CNN
+F 2 "Resistor_SMD:R_0603_1608Metric" V 6480 1900 50  0001 C CNN
 F 3 "~" H 6550 1900 50  0001 C CNN
 	1    6550 1900
@@
 F 0 "C17" H 6415 2196 50  0000 L CNN
 F 1 "1n" H 6415 2105 50  0000 L CNN
-F 2 "" H 6338 2000 50  0001 C CNN
+F 2 "Capacitor_SMD:C_0603_1608Metric" H 6338 2000 50  0001 C CNN
 F 3 "~" H 6300 2150 50  0001 C CNN
 	1    6300 2150
@@
 F 0 "C16" H 5765 2496 50  0000 L CNN
 F 1 "100n" H 5765 2405 50  0000 L CNN
-F 2 "" H 5688 2300 50  0001 C CNN
+F 2 "Capacitor_SMD:C_0603_1608Metric" H 5688 2300 50  0001 C CNN
 F 3 "~" H 5650 2450 50  0001 C CNN
 	1    5650 2450
@@
 F 0 "R28" H 8870 1546 50  0000 L CNN
 F 1 "24K" H 8870 1455 50  0000 L CNN
-F 2 "" V 8730 1500 50  0001 C CNN
+F 2 "Resistor_SMD:R_0603_1608Metric" V 8730 1500 50  0001 C CNN
 F 3 "~" H 8800 1500 50  0001 C CNN
 	1    8800 1500
@@
 F 0 "R29" H 8870 2546 50  0000 L CNN
 F 1 "620" H 8870 2455 50  0000 L CNN
-F 2 "" V 8730 2500 50  0001 C CNN
+F 2 "Resistor_SMD:R_0603_1608Metric" V 8730 2500 50  0001 C CNN
 F 3 "~" H 8800 2500 50  0001 C CNN
 	1    8800 2500
@@
 F 0 "R27" V 8043 1950 50  0000 C CNN
 F 1 "750" V 8134 1950 50  0000 C CNN
-F 2 "" V 8180 1950 50  0001 C CNN
+F 2 "Resistor_SMD:R_0603_1608Metric" V 8180 1950 50  0001 C CNN
 F 3 "~" H 8250 1950 50  0001 C CNN
 	1    8250 1950
@@
 F 0 "C23" V 8348 1950 50  0000 C CNN
 F 1 "68nF" V 8439 1950 50  0000 C CNN
-F 2 "" H 8638 1800 50  0001 C CNN
+F 2 "Capacitor_SMD:C_0603_1608Metric" H 8638 1800 50  0001 C CNN
 F 3 "~" H 8600 1950 50  0001 C CNN
 	1    8600 1950
@@
 F 0 "C22" V 8148 2300 50  0000 C CNN
 F 1 "3.9nF" V 8239 2300 50  0000 C CNN
-F 2 "" H 8438 2150 50  0001 C CNN
+F 2 "Capacitor_SMD:C_0603_1608Metric" H 8438 2150 50  0001 C CNN
 F 3 "~" H 8400 2300 50  0001 C CNN
 	1    8400 2300
@@
 F 0 "C18" H 7400 1900 50  0000 L CNN
 F 1 "100n" H 7350 1650 50  0000 L CNN
-F 2 "" H 7388 1600 50  0001 C CNN
+F 2 "Capacitor_SMD:C_0603_1608Metric" H 7388 1600 50  0001 C CNN
 F 3 "~" H 7350 1750 50  0001 C CNN
 	1    7350 1750
@@
 F 0 "C20" H 7768 1796 50  0000 L CNN
 F 1 "4µ7" H 7768 1705 50  0000 L CNN
-F 2 "" H 7688 1600 50  0001 C CNN
+F 2 "Capacitor_THT:CP_Radial_D16.0mm_P7.50mm" H 7688 1600 50  0001 C CNN
 F 3 "~" H 7650 1750 50  0001 C CNN
 	1    7650 1750
@@
 F 0 "C25" H 9168 1746 50  0000 L CNN
 F 1 "470µ" H 9100 1600 50  0000 L CNN
-F 2 "" H 9088 1550 50  0001 C CNN
+F 2 "Capacitor_THT:CP_Radial_D16.0mm_P7.50mm" H 9088 1550 50  0001 C CNN
 F 3 "~" H 9050 1700 50  0001 C CNN
 	1    9050 1700
@@
 F 0 "C27" H 9518 1746 50  0000 L CNN
 F 1 "470µ" H 9450 1600 50  0000 L CNN
-F 2 "" H 9438 1550 50  0001 C CNN
+F 2 "Capacitor_THT:CP_Radial_D16.0mm_P7.50mm" H 9438 1550 50  0001 C CNN
 F 3 "~" H 9400 1700 50  0001 C CNN
 	1    9400 1700
@@
 F 0 "C29" H 9868 1746 50  0000 L CNN
 F 1 "470µ" H 9800 1600 50  0000 L CNN
-F 2 "" H 9788 1550 50  0001 C CNN
+F 2 "Capacitor_THT:CP_Radial_D16.0mm_P7.50mm" H 9788 1550 50  0001 C CNN
 F 3 "~" H 9750 1700 50  0001 C CNN
 	1    9750 1700
@@
 F 0 "C30" H 10218 1746 50  0000 L CNN
 F 1 "470µ" H 10150 1600 50  0000 L CNN
-F 2 "" H 10138 1550 50  0001 C CNN
+F 2 "Capacitor_THT:CP_Radial_D16.0mm_P7.50mm" H 10138 1550 50  0001 C CNN
 F 3 "~" H 10100 1700 50  0001 C CNN
 	1    10100 1700
@@
 F 0 "C14" H 3865 1846 50  0000 L CNN
 F 1 "100n" H 3865 1755 50  0000 L CNN
-F 2 "" H 3788 1650 50  0001 C CNN
+F 2 "Capacitor_SMD:C_0603_1608Metric" H 3788 1650 50  0001 C CNN
 F 3 "~" H 3750 1800 50  0001 C CNN
 	1    3750 1800
@@
 F 0 "C13" H 3468 1846 50  0000 L CNN
 F 1 "470µ" H 3468 1755 50  0000 L CNN
-F 2 "" H 3388 1650 50  0001 C CNN
+F 2 "Capacitor_THT:CP_Radial_D16.0mm_P7.50mm" H 3388 1650 50  0001 C CNN
 F 3 "~" H 3350 1800 50  0001 C CNN
 	1    3350 1800
@@
 F 0 "C12" H 3118 1846 50  0000 L CNN
 F 1 "470µ" H 3118 1755 50  0000 L CNN
-F 2 "" H 3038 1650 50  0001 C CNN
+F 2 "Capacitor_THT:CP_Radial_D16.0mm_P7.50mm" H 3038 1650 50  0001 C CNN
 F 3 "~" H 3000 1800 50  0001 C CNN
 	1    3000 1800
@@
 F 0 "R24" V 6050 1650 50  0000 C CNN
 F 1 "3K6" V 5950 1650 50  0000 C CNN
-F 2 "" V 5980 1650 50  0001 C CNN
+F 2 "Resistor_SMD:R_0603_1608Metric" V 5980 1650 50  0001 C CNN
 F 3 "~" H 6050 1650 50  0001 C CNN
 	1    6050 1650
@@
 F 0 "D2" H 7050 984 50  0000 C CNN
 F 1 "D_Schottky" H 7050 1075 50  0000 C CNN
-F 2 "" H 7050 1200 50  0001 C CNN
+F 2 "Diode_SMD:D_1206_3216Metric" H 7050 1200 50  0001 C CNN
 F 3 "~" H 7050 1200 50  0001 C CNN
 	1    7050 1200
@@
 F 0 "C19" H 7518 4046 50  0000 L CNN
 F 1 "10u" H 7518 3955 50  0000 L CNN
-F 2 "" H 7438 3850 50  0001 C CNN
+F 2 "Capacitor_SMD:CP_Elec_4x3.9" H 7438 3850 50  0001 C CNN
 F 3 "~" H 7400 4000 50  0001 C CNN
 	1    7400 4000
@@
 F 0 "C21" H 7865 4046 50  0000 L CNN
 F 1 "100n" H 7865 3955 50  0000 L CNN
-F 2 "" H 7788 3850 50  0001 C CNN
+F 2 "Capacitor_SMD:C_0603_1608Metric" H 7788 3850 50  0001 C CNN
 F 3 "~" H 7750 4000 50  0001 C CNN
 	1    7750 4000
@@
 F 0 "C24" H 9015 4046 50  0000 L CNN
 F 1 "10u" H 9015 3955 50  0000 L CNN
-F 2 "" H 8938 3850 50  0001 C CNN
+F 2 "Capacitor_SMD:C_1206_3216Metric" H 8938 3850 50  0001 C CNN
 F 3 "~" H 8900 4000 50  0001 C CNN
 	1    8900 4000
@@
 F 0 "C28" H 9765 4046 50  0000 L CNN
 F 1 "100n" H 9765 3955 50  0000 L CNN
-F 2 "" H 9688 3850 50  0001 C CNN
+F 2 "Capacitor_SMD:C_0603_1608Metric" H 9688 3850 50  0001 C CNN
 F 3 "~" H 9650 4000 50  0001 C CNN
 	1    9650 4000
@@
 F 0 "C31" H 10915 4046 50  0000 L CNN
 F 1 "10u" H 10915 3955 50  0000 L CNN
-F 2 "" H 10838 3850 50  0001 C CNN
+F 2 "Capacitor_SMD:C_1206_3216Metric" H 10838 3850 50  0001 C CNN
 F 3 "~" H 10800 4000 50  0001 C CNN
 	1    10800 4000
@@
 F 0 "R18" H 2000 1450 50  0000 R CNN
 F 1 "10K" H 2050 1550 50  0000 R CNN
-F 2 "" V 1780 1500 50  0001 C CNN
+F 2 "Resistor_SMD:R_0603_1608Metric" V 1780 1500 50  0001 C CNN
 F 3 "~" H 1850 1500 50  0001 C CNN
 	1    1850 1500
@@
 F 0 "TP7" H 2758 1370 50  0000 L CNN
 F 1 "TestPoint" H 2758 1279 50  0000 L CNN
-F 2 "" H 2900 1250 50  0001 C CNN
+F 2 "TestPoint:TestPoint_Pad_2.5x2.5mm" H 2900 1250 50  0001 C CNN
 F 3 "~" H 2900 1250 50  0001 C CNN
 	1    2700 1250
@@
 F 0 "Q2" H 4005 3046 50  0000 L CNN
 F 1 "Q_NMOS_GDS" H 4005 2955 50  0000 L CNN
-F 2 "" H 4000 3100 50  0001 C CNN
+F 2 "FE Footprints:SOT-23" H 4000 3100 50  0001 C CNN
 F 3 "~" H 3800 3000 50  0001 C CNN
 	1    3800 3000
@@
 F 0 "Q1" H 3405 3446 50  0000 L CNN
 F 1 "Q_NMOS_GDS" H 3405 3355 50  0000 L CNN
-F 2 "" H 3400 3500 50  0001 C CNN
+F 2 "FE Footprints:SOT-23" H 3400 3500 50  0001 C CNN
 F 3 "~" H 3200 3400 50  0001 C CNN
 	1    3200 3400
@@
 F 0 "R19" H 3370 2846 50  0000 L CNN
 F 1 "1K" H 3370 2755 50  0000 L CNN
-F 2 "" V 3230 2800 50  0001 C CNN
+F 2 "Resistor_SMD:R_0603_1608Metric" V 3230 2800 50  0001 C CNN
 F 3 "~" H 3300 2800 50  0001 C CNN
 	1    3300 2800
