File: uc.sch (KiCad schematic (older format))
At the start: 42 parts, among them J1 AVR-ISP-6, J2 AVR-ISP-6, U1 MAX481E, U2 ATmega328P-AU, U3 ATmega328P-AU, Y1 Crystal, Y2 Crystal

Commit message: started assigning footprints
Parts:
- C1, C10, C11, C2, C3, C4, C5, C6, C7, C8, C9: footprint (none) -> Capacitor_SMD:C_0603_1608Metric
- D1: footprint (none) -> LED_SMD:LED_Cree-PLCC4_5x5mm_CW
- J1, J2: footprint (none) -> Connector_IDC:IDC-Header_2x03_P2.54mm_Vertical
- R1, R10, R11, R12, R13, R14, R15, R16, R17, R2, R3, R4, R5, R6, R7, R8, R9: footprint (none) -> Resistor_SMD:R_0603_1608Metric
- TP1, TP2, TP3, TP4, TP5, TP6: footprint (none) -> TestPoint:TestPoint_Pad_2.5x2.5mm
- U1: footprint (none) -> Package_SO:SOIC-8_3.9x4.9mm_P1.27mm
Changed lines of the file:
@@
 F 0 "J2" H 9720 1654 50  0000 R CNN
 F 1 "AVR-ISP-6" H 9720 1745 50  0000 R CNN
-F 2 "" V 9750 1700 50  0001 C CNN
+F 2 "Connector_IDC:IDC-Header_2x03_P2.54mm_Vertical" V 9750 1700 50  0001 C CNN
 F 3 " ~" H 8725 1100 50  0001 C CNN
 	1    10000 1650
@@
 F 0 "J1" H 8120 1654 50  0000 R CNN
 F 1 "AVR-ISP-6" H 8120 1745 50  0000 R CNN
-F 2 "" V 8150 1700 50  0001 C CNN
+F 2 "Connector_IDC:IDC-Header_2x03_P2.54mm_Vertical" V 8150 1700 50  0001 C CNN
 F 3 " ~" H 7125 1100 50  0001 C CNN
 	1    8400 1650
@@
 F 0 "C10" H 9915 4246 50  0000 L CNN
 F 1 "22p" H 9915 4155 50  0000 L CNN
-F 2 "" H 9838 4050 50  0001 C CNN
+F 2 "Capacitor_SMD:C_0603_1608Metric" H 9838 4050 50  0001 C CNN
 F 3 "~" H 9800 4200 50  0001 C CNN
 	1    9800 4200
@@
 F 0 "C11" H 10365 4246 50  0000 L CNN
 F 1 "22p" H 10365 4155 50  0000 L CNN
-F 2 "" H 10288 4050 50  0001 C CNN
+F 2 "Capacitor_SMD:C_0603_1608Metric" H 10288 4050 50  0001 C CNN
 F 3 "~" H 10250 4200 50  0001 C CNN
 	1    10250 4200
@@
 F 0 "R17" V 9243 4700 50  0000 C CNN
 F 1 "10K" V 9334 4700 50  0000 C CNN
-F 2 "" V 9380 4700 50  0001 C CNN
+F 2 "Resistor_SMD:R_0603_1608Metric" V 9380 4700 50  0001 C CNN
 F 3 "~" H 9450 4700 50  0001 C CNN
 	1    9450 4700
@@
 F 0 "C8" H 9115 2846 50  0000 L CNN
 F 1 "100n" H 9115 2755 50  0000 L CNN
-F 2 "" H 9038 2650 50  0001 C CNN
+F 2 "Capacitor_SMD:C_0603_1608Metric" H 9038 2650 50  0001 C CNN
 F 3 "~" H 9000 2800 50  0001 C CNN
 	1    9000 2800
@@
 F 0 "C9" H 9515 2846 50  0000 L CNN
 F 1 "10µ" H 9515 2755 50  0000 L CNN
-F 2 "" H 9438 2650 50  0001 C CNN
+F 2 "Capacitor_SMD:C_0603_1608Metric" H 9438 2650 50  0001 C CNN
 F 3 "~" H 9400 2800 50  0001 C CNN
 	1    9400 2800
@@
 F 0 "C1" H 2015 4096 50  0000 L CNN
 F 1 "22p" H 2015 4005 50  0000 L CNN
-F 2 "" H 1938 3900 50  0001 C CNN
+F 2 "Capacitor_SMD:C_0603_1608Metric" H 1938 3900 50  0001 C CNN
 F 3 "~" H 1900 4050 50  0001 C CNN
 	1    1900 4050
@@
 F 0 "C2" H 2465 4096 50  0000 L CNN
 F 1 "22p" H 2465 4005 50  0000 L CNN
-F 2 "" H 2388 3900 50  0001 C CNN
+F 2 "Capacitor_SMD:C_0603_1608Metric" H 2388 3900 50  0001 C CNN
 F 3 "~" H 2350 4050 50  0001 C CNN
 	1    2350 4050
@@
 F 0 "R8" V 4743 4650 50  0000 C CNN
 F 1 "10K" V 4834 4650 50  0000 C CNN
-F 2 "" V 4880 4650 50  0001 C CNN
+F 2 "Resistor_SMD:R_0603_1608Metric" V 4880 4650 50  0001 C CNN
 F 3 "~" H 4950 4650 50  0001 C CNN
 	1    4950 4650
@@
 F 0 "C6" H 4615 2796 50  0000 L CNN
 F 1 "100n" H 4615 2705 50  0000 L CNN
-F 2 "" H 4538 2600 50  0001 C CNN
+F 2 "Capacitor_SMD:C_0603_1608Metric" H 4538 2600 50  0001 C CNN
 F 3 "~" H 4500 2750 50  0001 C CNN
 	1    4500 2750
@@
 F 0 "C7" H 5015 2796 50  0000 L CNN
 F 1 "10µ" H 5015 2705 50  0000 L CNN
-F 2 "" H 4938 2600 50  0001 C CNN
+F 2 "Capacitor_SMD:C_0603_1608Metric" H 4938 2600 50  0001 C CNN
 F 3 "~" H 4900 2750 50  0001 C CNN
 	1    4900 2750
@@
 F 0 "R9" H 5130 3504 50  0000 R CNN
 F 1 "10K" H 5130 3595 50  0000 R CNN
-F 2 "" V 5130 3550 50  0001 C CNN
+F 2 "Resistor_SMD:R_0603_1608Metric" V 5130 3550 50  0001 C CNN
 F 3 "~" H 5200 3550 50  0001 C CNN
 	1    5200 3550
@@
 F 0 "R13" H 5430 3504 50  0000 R CNN
 F 1 "10K" H 5430 3595 50  0000 R CNN
-F 2 "" V 5430 3550 50  0001 C CNN
+F 2 "Resistor_SMD:R_0603_1608Metric" V 5430 3550 50  0001 C CNN
 F 3 "~" H 5500 3550 50  0001 C CNN
 	1    5500 3550
@@
 F 0 "R10" H 5230 5304 50  0000 R CNN
 F 1 "10K" H 5230 5395 50  0000 R CNN
-F 2 "" V 5230 5350 50  0001 C CNN
+F 2 "Resistor_SMD:R_0603_1608Metric" V 5230 5350 50  0001 C CNN
 F 3 "~" H 5300 5350 50  0001 C CNN
 	1    5300 5350
@@
 F 0 "D1" V 6996 4520 50  0000 R CNN
 F 1 "LED_ARGB" V 6905 4520 50  0000 R CNN
-F 2 "" H 6950 4800 50  0001 C CNN
+F 2 "LED_SMD:LED_Cree-PLCC4_5x5mm_CW" H 6950 4800 50  0001 C CNN
 F 3 "~" H 6950 4800 50  0001 C CNN
 	1    6950 4850
@@
 F 0 "R14" V 6450 5200 50  0000 C CNN
 F 1 "520" V 6400 5000 50  0000 C CNN
-F 2 "" V 6380 5200 50  0001 C CNN
+F 2 "Resistor_SMD:R_0603_1608Metric" V 6380 5200 50  0001 C CNN
 F 3 "~" H 6450 5200 50  0001 C CNN
 	1    6450 5200
@@
 F 0 "R15" V 6450 5300 50  0000 C CNN
 F 1 "520" V 6400 5100 50  0000 C CNN
-F 2 "" V 6380 5300 50  0001 C CNN
+F 2 "Resistor_SMD:R_0603_1608Metric" V 6380 5300 50  0001 C CNN
 F 3 "~" H 6450 5300 50  0001 C CNN
 	1    6450 5300
@@
 F 0 "R16" V 6450 5400 50  0000 C CNN
 F 1 "520" V 6400 5200 50  0000 C CNN
-F 2 "" V 6380 5400 50  0001 C CNN
+F 2 "Resistor_SMD:R_0603_1608Metric" V 6380 5400 50  0001 C CNN
 F 3 "~" H 6450 5400 50  0001 C CNN
 	1    6450 5400
@@
 F 0 "TP3" V 5100 6100 50  0000 L CNN
 F 1 "TestPoint" V 5150 6300 50  0000 L CNN
-F 2 "" H 5350 6100 50  0001 C CNN
+F 2 "TestPoint:TestPoint_Pad_2.5x2.5mm" H 5350 6100 50  0001 C CNN
 F 3 "~" H 5350 6100 50  0001 C CNN
 	1    5150 6100
@@
 F 0 "TP4" V 5100 6250 50  0000 L CNN
 F 1 "TestPoint" V 5150 6450 50  0000 L CNN
-F 2 "" H 5350 6250 50  0001 C CNN
+F 2 "TestPoint:TestPoint_Pad_2.5x2.5mm" H 5350 6250 50  0001 C CNN
 F 3 "~" H 5350 6250 50  0001 C CNN
 	1    5150 6250
@@
 F 0 "TP5" V 5100 6400 50  0000 L CNN
 F 1 "TestPoint" V 5150 6600 50  0000 L CNN
-F 2 "" H 5350 6400 50  0001 C CNN
+F 2 "TestPoint:TestPoint_Pad_2.5x2.5mm" H 5350 6400 50  0001 C CNN
 F 3 "~" H 5350 6400 50  0001 C CNN
 	1    5150 6400
@@
 F 0 "TP6" V 5100 6550 50  0000 L CNN
 F 1 "TestPoint" V 5150 6750 50  0000 L CNN
-F 2 "" H 5350 6550 50  0001 C CNN
+F 2 "TestPoint:TestPoint_Pad_2.5x2.5mm" H 5350 6550 50  0001 C CNN
 F 3 "~" H 5350 6550 50  0001 C CNN
 	1    5150 6550
@@
 F 0 "C5" H 2915 1646 50  0000 L CNN
 F 1 "10µ" H 2850 1500 50  0000 L CNN
-F 2 "" H 2838 1450 50  0001 C CNN
+F 2 "Capacitor_SMD:C_0603_1608Metric" H 2838 1450 50  0001 C CNN
 F 3 "~" H 2800 1600 50  0001 C CNN
 	1    2800 1600
@@
 F 0 "C3" H 2565 1646 50  0000 L CNN
 F 1 "100n" H 2500 1500 50  0000 L CNN
-F 2 "" H 2488 1450 50  0001 C CNN
+F 2 "Capacitor_SMD:C_0603_1608Metric" H 2488 1450 50  0001 C CNN
 F 3 "~" H 2450 1600 50  0001 C CNN
 	1    2450 1600
@@
 F 0 "R11" V 5450 4850 50  0000 C CNN
 F 1 "100" V 5400 5050 50  0000 C CNN
-F 2 "" V 5380 4850 50  0001 C CNN
+F 2 "Resistor_SMD:R_0603_1608Metric" V 5380 4850 50  0001 C CNN
 F 3 "~" H 5450 4850 50  0001 C CNN
 	1    5450 4850
@@
 F 0 "R12" V 5450 4950 50  0000 C CNN
 F 1 "100" V 5500 5150 50  0000 C CNN
-F 2 "" V 5380 4950 50  0001 C CNN
+F 2 "Resistor_SMD:R_0603_1608Metric" V 5380 4950 50  0001 C CNN
 F 3 "~" H 5450 4950 50  0001 C CNN
 	1    5450 4950
@@
 F 0 "C4" H 2865 3446 50  0000 L CNN
 F 1 "100n" H 2865 3355 50  0000 L CNN
-F 2 "" H 2788 3250 50  0001 C CNN
+F 2 "Capacitor_SMD:C_0603_1608Metric" H 2788 3250 50  0001 C CNN
 F 3 "~" H 2750 3400 50  0001 C CNN
 	1    2750 3400
@@
 F 0 "TP1" V 2800 1950 50  0000 L CNN
 F 1 "TestPoint" V 2850 2150 50  0000 L CNN
-F 2 "" H 3050 1950 50  0001 C CNN
+F 2 "TestPoint:TestPoint_Pad_2.5x2.5mm" H 3050 1950 50  0001 C CNN
 F 3 "~" H 3050 1950 50  0001 C CNN
 	1    2850 1950
@@
 F 0 "TP2" V 2800 2500 50  0000 L CNN
 F 1 "TestPoint" V 2850 2700 50  0000 L CNN
-F 2 "" H 3050 2500 50  0001 C CNN
+F 2 "TestPoint:TestPoint_Pad_2.5x2.5mm" H 3050 2500 50  0001 C CNN
 F 3 "~" H 3050 2500 50  0001 C CNN
 	1    2850 2500
@@
 F 0 "R2" H 1350 1550 50  0000 R CNN
 F 1 "10K" H 1400 1850 50  0000 R CNN
-F 2 "" V 1180 1700 50  0001 C CNN
+F 2 "Resistor_SMD:R_0603_1608Metric" V 1180 1700 50  0001 C CNN
 F 3 "~" H 1250 1700 50  0001 C CNN
 	1    1250 1700
@@
 F 0 "R3" H 1500 1550 50  0000 R CNN
 F 1 "10K" H 1550 1850 50  0000 R CNN
-F 2 "" V 1330 1700 50  0001 C CNN
+F 2 "Resistor_SMD:R_0603_1608Metric" V 1330 1700 50  0001 C CNN
 F 3 "~" H 1400 1700 50  0001 C CNN
 	1    1400 1700
@@
 F 0 "R4" H 1650 1550 50  0000 R CNN
 F 1 "10K" H 1700 1850 50  0000 R CNN
-F 2 "" V 1480 1700 50  0001 C CNN
+F 2 "Resistor_SMD:R_0603_1608Metric" V 1480 1700 50  0001 C CNN
 F 3 "~" H 1550 1700 50  0001 C CNN
 	1    1550 1700
@@
 F 0 "U1" H 2000 2828 50  0000 C CNN
 F 1 "MAX481E" H 2000 2737 50  0000 C CNN
-F 2 "" H 2000 1450 50  0001 C CNN
+F 2 "Package_SO:SOIC-8_3.9x4.9mm_P1.27mm" H 2000 1450 50  0001 C CNN
 F 3 "https://datasheets.maximintegrated.com/en/ds/MAX1487E-MAX491E.pdf" H 2000 2200 50  0001 C CNN
 	1    2000 2150
@@
 F 0 "R1" H 1200 1550 50  0000 R CNN
 F 1 "10K" H 1250 1850 50  0000 R CNN
-F 2 "" V 1030 1700 50  0001 C CNN
+F 2 "Resistor_SMD:R_0603_1608Metric" V 1030 1700 50  0001 C CNN
 F 3 "~" H 1100 1700 50  0001 C CNN
 	1    1100 1700
@@
 F 0 "R5" H 2750 2050 50  0000 R CNN
 F 1 "120" H 2850 2250 50  0000 R CNN
-F 2 "" V 2580 2200 50  0001 C CNN
+F 2 "Resistor_SMD:R_0603_1608Metric" V 2580 2200 50  0001 C CNN
 F 3 "~" H 2650 2200 50  0001 C CNN
 	1    2650 2200
@@
 F 0 "R7" V 3100 2300 50  0000 R CNN
 F 1 "22K" V 3200 2300 50  0000 R CNN
-F 2 "" V 3030 2250 50  0001 C CNN
+F 2 "Resistor_SMD:R_0603_1608Metric" V 3030 2250 50  0001 C CNN
 F 3 "~" H 3100 2250 50  0001 C CNN
 	1    3100 2250
@@
 F 0 "R6" V 2650 2600 50  0000 R CNN
 F 1 "22K" V 2750 2600 50  0000 R CNN
-F 2 "" V 2580 2550 50  0001 C CNN
+F 2 "Resistor_SMD:R_0603_1608Metric" V 2580 2550 50  0001 C CNN
 F 3 "~" H 2650 2550 50  0001 C CNN
 	1    2650 2550
